File: Base roulante/Base roulante.kicad_sch (KiCad schematic)
At the start: 15 parts, among them J1 RJ_can, J2 RJ_can, J5 connector_power, U1 Blue Pill, U2 MCP2551-I-SN

Commit message: Update base roulante
Parts:
- C1: footprint (none) -> Capacitor_THT:CP_Radial_D5.0mm_P2.00mm
- D+5V1: value (none) -> LED; footprint (none) -> LED_THT:LED_D5.0mm
- R1, R2: footprint (none) -> Resistor_SMD:R_0805_2012Metric
- RC_Droite1: value (none) -> roues_codeuses
Connections:
- net A_D: now also U1.31 (PA6); no longer U1.25 (PA0)
- net B_D: now also U1.32 (PA7); no longer U1.26 (PA1)
- net DIR_D: now also U1.2 (PB13); no longer U1.31 (PA6)
- net DIR_G: now also U1.1 (PB12); no longer U1.32 (PA7)
- net PWM_D: now also U1.6 (PA9); no longer U1.33 (PB0)
- net PWM_G: now also U1.5 (PA8); no longer U1.34 (PB1)
Changed lines of the file:
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@@
     )
   )
-  (global_label "PWM_D" (shape input) (at 77.47 92.71 0) (fields_autoplaced)
-    (effects (font (size 1.27 1.27)) (justify left))
-    (property "Références Inter-Feuilles" "${INTERSHEET_REFS}" (id 0) (at 86.2936 92.6306 0)
-      (effects (font (size 1.27 1.27)) (justify left) hide)
+  (global_label "PWM_D" (shape input) (at 36.83 95.25 180) (fields_autoplaced)
+    (effects (font (size 1.27 1.27)) (justify right))
+    (property "Références Inter-Feuilles" "${INTERSHEET_REFS}" (id 0) (at 28.0064 95.3294 0)
+      (effects (font (size 1.27 1.27)) (justify right) hide)
     )
   )
@@
     )
   )
-  (global_label "DIR_D" (shape input) (at 77.47 97.79 0) (fields_autoplaced)
-    (effects (font (size 1.27 1.27)) (justify left))
-    (property "Références Inter-Feuilles" "${INTERSHEET_REFS}" (id 0) (at 85.2655 97.7106 0)
-      (effects (font (size 1.27 1.27)) (justify left) hide)
+  (global_label "DIR_D" (shape input) (at 36.83 85.09 180) (fields_autoplaced)
+    (effects (font (size 1.27 1.27)) (justify right))
+    (property "Références Inter-Feuilles" "${INTERSHEET_REFS}" (id 0) (at 29.0345 85.1694 0)
+      (effects (font (size 1.27 1.27)) (justify right) hide)
     )
   )
@@
     )
   )
-  (global_label "DIR_G" (shape input) (at 77.47 95.25 0) (fields_autoplaced)
-    (effects (font (size 1.27 1.27)) (justify left))
-    (property "Références Inter-Feuilles" "${INTERSHEET_REFS}" (id 0) (at 85.2655 95.1706 0)
-      (effects (font (size 1.27 1.27)) (justify left) hide)
+  (global_label "DIR_G" (shape input) (at 36.83 82.55 180) (fields_autoplaced)
+    (effects (font (size 1.27 1.27)) (justify right))
+    (property "Références Inter-Feuilles" "${INTERSHEET_REFS}" (id 0) (at 29.0345 82.6294 0)
+      (effects (font (size 1.27 1.27)) (justify right) hide)
     )
   )
@@
     )
   )
-  (global_label "PWM_G" (shape input) (at 77.47 90.17 0) (fields_autoplaced)
-    (effects (font (size 1.27 1.27)) (justify left))
-    (property "Références Inter-Feuilles" "${INTERSHEET_REFS}" (id 0) (at 86.2936 90.0906 0)
-      (effects (font (size 1.27 1.27)) (justify left) hide)
+  (global_label "PWM_G" (shape input) (at 36.83 92.71 180) (fields_autoplaced)
+    (effects (font (size 1.27 1.27)) (justify right))
+    (property "Références Inter-Feuilles" "${INTERSHEET_REFS}" (id 0) (at 28.0064 92.7894 0)
+      (effects (font (size 1.27 1.27)) (justify right) hide)
     )
   )
@@
     )
   )
-  (global_label "B_D" (shape input) (at 77.47 110.49 0) (fields_autoplaced)
-    (effects (font (size 1.27 1.27)) (justify left))
-    (property "Références Inter-Feuilles" "${INTERSHEET_REFS}" (id 0) (at 83.3907 110.4106 0)
+  (global_label "B_D" (shape input) (at 77.47 95.25 0) (fields_autoplaced)
+    (effects (font (size 1.27 1.27)) (justify left))
+    (property "Références Inter-Feuilles" "${INTERSHEET_REFS}" (id 0) (at 83.3907 95.1706 0)
       (effects (font (size 1.27 1.27)) (justify left) hide)
     )
@@
     )
   )
-  (global_label "A_D" (shape input) (at 77.47 113.03 0) (fields_autoplaced)
-    (effects (font (size 1.27 1.27)) (justify left))
-    (property "Références Inter-Feuilles" "${INTERSHEET_REFS}" (id 0) (at 83.2093 112.9506 0)
+  (global_label "A_D" (shape input) (at 77.47 97.79 0) (fields_autoplaced)
+    (effects (font (size 1.27 1.27)) (justify left))
+    (property "Références Inter-Feuilles" "${INTERSHEET_REFS}" (id 0) (at 83.2093 97.7106 0)
       (effects (font (size 1.27 1.27)) (justify left) hide)
     )
@@
       (effects (font (size 1.27 1.27)) (justify left))
     )
-    (property "Footprint" "" (id 2) (at 92.202 41.91 90)
+    (property "Footprint" "Resistor_SMD:R_0805_2012Metric" (id 2) (at 92.202 41.91 90)
       (effects (font (size 1.27 1.27)) hide)
     )
@@
       (effects (font (size 1.27 1.27)) hide)
     )
-    (property "Value" "" (id 1) (at 172.72 111.7599 90)
+    (property "Value" "GND" (id 1) (at 172.72 111.7599 90)
       (effects (font (size 1.27 1.27)) (justify right))
     )
@@
       (effects (font (size 1.27 1.27)) hide)
     )
-    (property "Value" "" (id 1) (at 54.61 69.85 0))
+    (property "Value" "+5V" (id 1) (at 54.61 69.85 0))
     (property "Footprint" "" (id 2) (at 54.61 74.93 0)
       (effects (font (size 1.27 1.27)) hide)
@@
     (property "Reference" "R2" (id 0) (at 132.08 46.99 90))
     (property "Value" "R" (id 1) (at 132.08 44.45 90))
-    (property "Footprint" "" (id 2) (at 132.08 38.862 90)
+    (property "Footprint" "Resistor_SMD:R_0805_2012Metric" (id 2) (at 132.08 38.862 90)
       (effects (font (size 1.27 1.27)) hide)
     )
@@
       (effects (font (size 1.27 1.27)) (justify right))
     )
-    (property "Value" "" (id 1) (at 97.79 34.6074 90)
-      (effects (font (size 1.27 1.27)) (justify right))
-    )
-    (property "Footprint" "" (id 2) (at 93.98 31.75 0)
+    (property "Value" "LED" (id 1) (at 97.79 34.6074 90)
+      (effects (font (size 1.27 1.27)) (justify right))
+    )
+    (property "Footprint" "LED_THT:LED_D5.0mm" (id 2) (at 93.98 31.75 0)
       (effects (font (size 1.27 1.27)) hide)
     )
@@
       (effects (font (size 1.27 1.27)) hide)
     )
-    (property "Value" "" (id 1) (at 173.99 81.2799 90)
+    (property "Value" "GND" (id 1) (at 173.99 81.2799 90)
       (effects (font (size 1.27 1.27)) (justify right))
     )
@@
       (effects (font (size 1.27 1.27)) hide)
     )
-    (property "Value" "" (id 1) (at 173.99 83.8199 90)
+    (property "Value" "+5V" (id 1) (at 173.99 83.8199 90)
       (effects (font (size 1.27 1.27)) (justify left))
     )
@@
       (effects (font (size 1.27 1.27)) hide)
     )
-    (property "Value" "" (id 1) (at 172.72 114.2999 90)
+    (property "Value" "+5V" (id 1) (at 172.72 114.2999 90)
       (effects (font (size 1.27 1.27)) (justify left))
     )
@@
       (effects (font (size 1.27 1.27)) hide)
     )
+    (pin "1")
     (pin "2")
     (pin "3")
     (pin "4")
-    (pin "1")
     (pin "5")
   )
@@
       (effects (font (size 1.27 1.27)) (justify left))
     )
-    (property "Footprint" "" (id 2) (at 108.9152 41.91 0)
+    (property "Footprint" "Capacitor_THT:CP_Radial_D5.0mm_P2.00mm" (id 2) (at 108.9152 41.91 0)
       (effects (font (size 1.27 1.27)) hide)
     )
@@
     (in_bom yes) (on_board yes) (fields_autoplaced)
     (property "Reference" "RC_Droite1" (id 0) (at 162.56 105.41 0))
-    (property "Value" "" (id 1) (at 162.56 107.95 0))
+    (property "Value" "roues_codeuses" (id 1) (at 162.56 107.95 0))
     (property "Footprint" "Robot:HE14-5-angle" (id 2) (at 168.91 109.22 0)
       (effects (font (size 1.27 1.27)) hide)
@@
       (effects (font (size 1.27 1.27)) hide)
     )
-    (property "Value" "" (id 1) (at 214.63 24.13 0))
+    (property "Value" "+12V" (id 1) (at 214.63 24.13 0))
     (property "Footprint" "" (id 2) (at 214.63 29.21 0)
       (effects (font (size 1.27 1.27)) hide)

Commit message: Add Base roulante updated
Parts:
- added C2: 470u, Capacitor_THT:CP_Radial_D5.0mm_P2.00mm, symbol Device:C_Polarized
- added DPANIC1: LED Rouge, LED_SMD:LED_0805_2012Metric, symbol Device:LED
- added R4: 330, Resistor_SMD:R_0805_2012Metric, symbol Device:R
- C1: value C_Polarized -> 47u
- D+12V1: value LED -> LED bleu; footprint LED_THT:LED_D5.0mm -> LED_SMD:LED_0805_2012Metric
- D+5V1: value LED -> LED Verte; footprint LED_THT:LED_D5.0mm -> LED_SMD:LED_0805_2012Metric
- R1: value R -> 330
- R2: value R -> 10k
- R3: value R -> 1k
Connections:
- net +12V: now also C2.1
- net GND: now also C2.2, DPANIC1.1 (K)
- net PANIC: now reaches U1.16 (PB8)
- net PANIC: now also DPANIC1.2 (A), R4.2
- net +3.3V: now reaches U1.20 (3V3)
- net +3.3V: now also U1.38 (3V3), R4.1
- no-connect marks 0 -> 26
Other:
- note added: "Panic"
- moved on the sheet: D+12V1, J5, Mot_Droit1, Mot_Gauche1, R3, RC_Droite1, RC_Gauche1, U1
