File: carteIO/testrobot.kicad_pcb (KiCad board)
At the start: 2 copper layers, 71.1 x 82.6 mm, 19 parts, among them J1 RJ_can, J2 RJ_can, J3 connector_power, U1 HC-SR04, U2 HC-SR04, U3 MCP2551-I-SN, U5 Nucleo_STM32G431KB

Commit message: carte IO
Other:
- board text added: "IO 2023-AAC Claudia & Joel"
- board text removed: "IO 2023-AAC"
Changed lines of the file:
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@@
     (effects (font (size 1 1) (thickness 0.15)) (justify left bottom))
   )
-  (gr_text "IO\n2023-AAC" (at 152.4 73.66) (layer "F.Cu")
+  (gr_text "IO\n2023-AAC\nClaudia & Joel" (at 163.83 74.93) (layer "F.Cu")
     (effects (font (size 1 1) (thickness 0.15)) (justify left bottom))
   )

Commit message: added some vias for the grownd plain
Routing:
- net Trig_b4: track 56.1 -> 61.1 mm, vias 1 -> 2
- net GND: vias 1 -> 8
- net Echo_b5: vias 1 -> 2
Changed lines of the file:
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@@
     (grid_origin 175.26 119.38)
     (pcbplotparams
-      (layerselection 0x00010fc_ffffffff)
+      (layerselection 0x0001000_ffffffff)
       (plot_on_all_layers_selection 0x0000000_00000000)
       (disableapertmacros false)
@@
       (outputformat 1)
       (mirror false)
-      (drillshape 1)
+      (drillshape 0)
       (scaleselection 1)
-      (outputdirectory "")
+      (outputdirectory "../fab/")
     )
   )
@@
     (fp_rect (start 14.351 -0.889) (end 16.129 36.449)
       (stroke (width 0.12) (type solid)) (fill none) (layer "F.SilkS"))
-    (fp_arc (start 3.967155 -10.260847) (mid 4.012928 -10.185275) (end 4.029561 -10.0985)
-      (stroke (width 0.12) (type solid)) (layer "F.SilkS"))
-    (fp_arc (start 4.151131 -10.424759) (mid 4.243692 -10.270872) (end 4.275977 -10.094215)
-      (stroke (width 0.12) (type solid)) (layer "F.SilkS"))
-    (fp_arc (start 4.625988 -10.535212) (mid 4.709181 -10.688645) (end 4.875989 -10.74)
+    (fp_arc (start 3.967155 -10.260847) (mid 4.01291 -10.185271) (end 4.029561 -10.0985)
+      (stroke (width 0.12) (type solid)) (layer "F.SilkS"))
+    (fp_arc (start 4.151131 -10.424759) (mid 4.243705 -10.270873) (end 4.275977 -10.094215)
+      (stroke (width 0.12) (type solid)) (layer "F.SilkS"))
+    (fp_arc (start 4.625988 -10.535212) (mid 4.709181 -10.688641) (end 4.875989 -10.74)
       (stroke (width 0.12) (type solid)) (layer "F.SilkS"))
     (fp_arc (start 4.625989 -10.391818) (mid 4.709183 -10.545247) (end 4.875989 -10.596605)
@@
     (fp_arc (start 10.922399 -10.090063) (mid 10.854026 -10.120573) (end 10.825988 -10.19)
       (stroke (width 0.12) (type solid)) (layer "F.SilkS"))
-    (fp_arc (start 11.176 -10.094215) (mid 11.208256 -10.27088) (end 11.300846 -10.424759)
-      (stroke (width 0.12) (type solid)) (layer "F.SilkS"))
-    (fp_arc (start 11.422416 -10.0985) (mid 11.439038 -10.18528) (end 11.484822 -10.260847)
+    (fp_arc (start 11.176 -10.094215) (mid 11.208251 -10.270884) (end 11.300846 -10.424759)
+      (stroke (width 0.12) (type solid)) (layer "F.SilkS"))
+    (fp_arc (start 11.422416 -10.0985) (mid 11.439043 -10.185276) (end 11.484822 -10.260847)
       (stroke (width 0.12) (type solid)) (layer "F.SilkS"))
     (fp_circle (center 5.969 28.067) (end 5.969001 28.067)
@@
   (segment (start 160.02 78.74) (end 185.42 78.74) (width 1) (layer "B.Cu") (net 1))
   (segment (start 160.02 83.82) (end 160.02 78.74) (width 1) (layer "B.Cu") (net 1))
+  (via (at 175.26 88.9) (size 0.8) (drill 0.4) (layers "F.Cu" "B.Cu") (free) (net 2))
+  (via (at 208.28 116.84) (size 0.8) (drill 0.4) (layers "F.Cu" "B.Cu") (free) (net 2))
   (via (at 210.82 129.54) (size 1) (drill 0.6) (layers "F.Cu" "B.Cu") (free) (net 2))
+  (via (at 157.48 101.6) (size 0.8) (drill 0.4) (layers "F.Cu" "B.Cu") (free) (net 2))
+  (via (at 185.42 76.2) (size 0.8) (drill 0.4) (layers "F.Cu" "B.Cu") (free) (net 2))
+  (via (at 203.2 147.32) (size 0.8) (drill 0.4) (layers "F.Cu" "B.Cu") (free) (net 2))
+  (via (at 190.5 101.6) (size 0.8) (drill 0.4) (layers "F.Cu" "B.Cu") (free) (net 2))
+  (via (at 152.4 144.78) (size 0.8) (drill 0.4) (layers "F.Cu" "B.Cu") (free) (net 2))
   (segment (start 215.9 127) (end 215.9 125.125) (width 1) (layer "F.Cu") (net 3))
   (segment (start 215.9 125.125) (end 216.565 124.46) (width 1) (layer "F.Cu") (net 3))
@@
   (segment (start 159.7425 128.905) (end 157.48 131.1675) (width 0.7) (layer "F.Cu") (net 25))
   (segment (start 170.18 111.76) (end 177.8 119.38) (width 1) (layer "F.Cu") (net 26))
-  (segment (start 177.8 119.38) (end 180.34 119.38) (width 1) (layer "F.Cu") (net 26))
+  (segment (start 177.8 119.38) (end 177.8 121.92) (width 1) (layer "F.Cu") (net 26))
+  (segment (start 177.8 121.92) (end 180.34 121.92) (width 1) (layer "F.Cu") (net 26))
+  (via (at 180.34 121.92) (size 0.8) (drill 0.4) (layers "F.Cu" "B.Cu") (net 26))
   (via (at 170.18 111.76) (size 1) (drill 0.6) (layers "F.Cu" "B.Cu") (net 26))
   (segment (start 167.64 109.22) (end 170.18 111.76) (width 1) (layer "B.Cu") (net 26))
@@
   (segment (start 170.18 111.76) (end 170.18 86.36) (width 1) (layer "B.Cu") (net 26))
   (segment (start 162.56 109.22) (end 167.64 109.22) (width 1) (layer "B.Cu") (net 26))
+  (segment (start 180.34 121.92) (end 180.34 119.38) (width 1) (layer "B.Cu") (net 26))
   (segment (start 167.64 101.6) (end 170.18 104.14) (width 1) (layer "F.Cu") (net 27))
   (segment (start 167.64 91.44) (end 167.64 101.6) (width 1) (layer "F.Cu") (net 27))
@@
   (segment (start 182.88 124.46) (end 185.42 121.92) (width 1) (layer "F.Cu") (net 28))
   (segment (start 185.42 121.92) (end 185.42 119.38) (width 1) (layer "F.Cu") (net 28))
-  (segment (start 182.88 116.84) (end 180.34 116.84) (width 1) (layer "F.Cu") (net 28))
   (segment (start 177.8 124.46) (end 182.88 124.46) (width 1) (layer "F.Cu") (net 28))
   (segment (start 167.64 114.3) (end 177.8 124.46) (width 1) (layer "F.Cu") (net 28))
   (via (at 167.64 114.3) (size 1) (drill 0.6) (layers "F.Cu" "B.Cu") (net 28))
+  (via (at 182.88 116.84) (size 0.8) (drill 0.4) (layers "F.Cu" "B.Cu") (net 28))
   (segment (start 165.1 111.76) (end 167.64 114.3) (width 1) (layer "B.Cu") (net 28))
   (segment (start 162.56 111.76) (end 165.1 111.76) (width 1) (layer "B.Cu") (net 28))
+  (segment (start 182.88 116.84) (end 180.34 116.84) (width 1) (layer "B.Cu") (net 28))
   (segment (start 169.545 128.905) (end 170.18 129.54) (width 0.7) (layer "F.Cu") (net 29))
   (segment (start 167.575 128.905) (end 169.545 128.905) (width 0.7) (layer "F.Cu") (net 29))
