File: Base_Roulante_2024/Base_Roulante_2024.kicad_sch (KiCad schematic)
At the start: 10 parts, among them J1 RJ_can, J2 RJ_can, U1 Nucleo_STM32G431KB, U2 MCP2551-I-SN, U3 DRV8811PWP, U4 DRV8811PWP

Commit message: Add files via upload
Parts:
- added U5, U6: DRV8811PWP, PWP28_5P18X3P1, symbol 2023-10-09_21-45-47:DRV8811PWP
Connections:
- net +5V: now also U1.27 (+5V)
- net CAN_RX: now also U1.5 (PA12)
- net CAN_TX: now also U1.13 (PA11)
- net GND: now also U1.29 (GND), U1.4 (GND)
Other:
- moved on the sheet: C1, D+5V1, J1, J2, R1, R2, U1, U2, U3, U4

Commit message: J'ai changé la carte Base Roulante pour n'avoir qu'un driver et des interfaces
Parts:
- removed C1: C_Polarized, Capacitor_THT:CP_Radial_D5.0mm_P2.00mm, symbol Device:C_Polarized
- removed D+5V1: LED, LED_THT:LED_D5.0mm, symbol Device:LED
- removed J1, J2: RJ_can, PCM_Robot:RJ12, symbol Robot:RJ_can
- removed R1, R2: R, Resistor_SMD:R_0805_2012Metric, symbol Device:R
- removed U1: Nucleo_STM32G431KB, Robot:Nucleo_STM32G431KB, symbol PCM_Robot:Nucleo_STM32G431KB
- removed U2: MCP2551-I-SN, Package_SO:SOIC-8_3.9x4.9mm_P1.27mm, symbol Interface_CAN_LIN:MCP2551-I-SN
- removed U4, U5, U6: DRV8811PWP, PWP28_5P18X3P1, symbol 2023-10-09_21-45-47:DRV8811PWP
- added C2: 10u, symbol Device:C
- added C3, C4, C5: 0.22u, symbol Device:C
- added C6, C7: C, symbol Device:C
- added C8: 0.1u, symbol Device:C
- added R: 82k, symbol Device:R
- added R10, R5, R9: 10k, symbol Device:R
- added R3, R4: 200m, symbol Device:R
- added R7, R8: R, symbol Device:R
Connections:
- net +5V: now also U3.10 (VCC), C2.1, R.1, R9.1
- net GND: now also U3.21 (GND), U3.29 (EPAD), U3.7 (GND), C2.2, C4.2, C6.2, C7.2, C8.2, R10.2, R3.1, R4.1, R5.2, R7.2, R8.2
- net at U3.1 (ISENA): now also R3.2
- net at U3.14 (ISENB): now also R4.2
- net +12V: now reaches U3.15 (VMB)
- net +12V: now also U3.28 (VMA), C5.1
- net CP1: now reaches U3.23 (CP1)
- net CP1: now also C3.2
- net CP2: now reaches U3.24 (CP2)
- net CP2: now also C3.1
- net at U3.8 (VREF): now also R.2, R5.1
- new net DECAY: C8.1, R10.1, R9.2
- new net RCA: C6.1, R7.1
- new net RCB: C7.1, R8.1
- new net VCP: C5.2
- new net VGD: C4.1
Other:
- note added: "Charge pump capacitor"
- note added: "If DECAY < 0.21*Vcc (Here 5V) then Fast decay If DECAY > 0.6*Vcc then Slow decay Otherwise Mixed Decay The capacitor fixed the timing the resistors fix the voltage divider hence the mode... Chose values from the datasheet example for now"
- note added: "Inputs to be provided digitally"
- note added: "Logic power supply Bypass Capacitor"
- note added: "Motor outputs to be provided with connector"
- note added: "Not connected"
- note added: "Output current range selection with Rsense = 0.1mOhm , and Max winding current = 0.35 A (Based on motor specs , a little over 0.31A per winding. Vref = 0.35 * 8 * Rsense = 0.35 * 8 * 0.2 = 0.56V So 10 k and 70 k voltage divider results in Vref = 0.625 V which is close enough"
- note added: "Pad thermique"
- note added: "Pins to configure stepping modes (Logic states) How to define the GND for these pins?"
- note added: "Toff (us) = R (Ohm) * C (nF) Tblank (ns) = 1400 (Ohm) * C (nF)"
- note added: "VMA and VMB are stepper motor PWR"
- note removed: "Bus CAN + Transceiver"
- note removed: "STM32 Nucleo"
- moved on the sheet: U3

Commit message: Update Base_Roulante_2024
Parts:
- removed U3: DRV8811PWP, PWP28_5P18X3P1, symbol 2023-10-09_21-45-47:DRV8811PWP
- added J2: Conn_01x06_Pin, symbol Connector:Conn_01x06_Pin
- added J3: Conn_01x08_Pin, symbol PCM_Robot:Conn_01x08_Pin
- added J5: connector_power, PCM_Robot:WR_TBL_3137_2pins, symbol Robot:connector_power
- added U1: DRV8811PWP, PWP28_5P18X3P1, symbol PCM_2023-10-09_21-45-47:DRV8811PWP
- C2, C3, C4, C5: footprint (none) -> Capacitor_SMD:C_0805_2012Metric_Pad1.18x1.45mm_HandSolder
- C6, C7: value C -> 1n; footprint (none) -> Capacitor_SMD:C_0805_2012Metric_Pad1.18x1.45mm_HandSolder
- R10, R3, R4, R9: footprint (none) -> Resistor_SMD:R_0805_2012Metric_Pad1.20x1.40mm_HandSolder
- R6: renamed from R; footprint (none) -> Resistor_SMD:R_0805_2012Metric_Pad1.20x1.40mm_HandSolder
- R7, R8: value R -> 47k; footprint (none) -> Resistor_SMD:R_0805_2012Metric_Pad1.20x1.40mm_HandSolder
Connections:
- net +12V: now also J5.1 (+12V), U1.15 (VMB), U1.28 (VMA)
- net +5V: now also J3.7 (Pin_7), U1.10 (VCC), U1.12 (USM1), U1.13 (USM0)
- net CP1: now also U1.23 (CP1)
- net CP2: now also U1.24 (CP2)
- net DECAY: now also U1.5 (DECAY)
- net DIR: now also J3.1 (Pin_1), U1.3 (DIR)
- net ENABLEN: now also J3.6 (Pin_6), U1.26 (ENABLEN)
- net GND: now also J3.2 (Pin_2), J5.2 (GND), U1.21 (GND), U1.29 (EPAD), U1.7 (GND)
- net HOMEn: now also U1.2 (HOME)
- net PhaseA_1: now also J2.1 (Pin_1), U1.4 (AOUT1)
- net PhaseA_2: now also J2.2 (Pin_2), U1.25 (AOUT2)
- net PhaseA_COM: now also J2.4 (Pin_4)
- net PhaseB_1: now also J2.5 (Pin_5), U1.11 (BOUT1)
- net PhaseB_2: now also J2.6 (Pin_6), U1.18 (BOUT2)
- net PhaseB_COM: now also J2.3 (Pin_3)
- net RCA: now also U1.6 (RCA)
- net RCB: now also U1.9 (RCB)
- net RESETN: now also J3.3 (Pin_3), U1.17 (RESETN)
- net SLEEPN: now also J3.5 (Pin_5), U1.27 (SLEEPN)
- net SRN: now also J3.4 (Pin_4), U1.16 (SRN)
- net STEP: now also J3.8 (Pin_8), U1.19 (STEP)
- net VCP: now also U1.22 (VCP)
- net VGD: now also U1.20 (VGD)
- net at R3.2: now also U1.1 (ISENA)
- net at R4.2: now also U1.14 (ISENB)
- net Vref: now reaches R5.1, R6.2
- net Vref: now also U1.8 (VREF)
- no-connect marks 0 -> 2
Other:
- note added: "0.0"
- note added: "29/10/2023"
- note added: "Driver Moteur Pas à pas"
- note added: "Errors are due to ISENB and ISENA being power inputs they should be regular inputs"
- note added: "INPUTS/OUTPUTS"
- note added: "J'ai choisi les valeurs dans la datasheet car on ne se sert pas de cette fonctionnalité. On pourrait changer les valeurs"
- note added: "MAIN DRIVER"
- note added: "No need for extra resistors, there are some already in the IC"
- note added: "POWER +12V"
- note added: "Placement de la terre pour prévenir des interferences entre step et dir"
- moved on the sheet: C8, R10, R9
